Commit message: updated cobotta configuration files

File: ROS2_ws/src/denso_cobotta_description/urdf/cobotta.urdf.xacro (robot description, xacro)
@@ -33,4 +33,9 @@
 		</plugin>
 	</gazebo>
+	<link name="world"/>
+	<joint name="joint_w" type="fixed">
+		<parent link="world"/>
+		<child link="base_link"/>
+	</joint>
 	<link name="base_link">
 		<visual>

Commit message: Demo pick and place package

File: ROS2_ws/src/denso_cobotta_description/urdf/cobotta.urdf.xacro (robot description, xacro)
@@ -80,14 +80,4 @@
 		<dynamics damping="${joint_damping}" friction="${joint_friction}" />
 	</joint>
-	<transmission name="trans_1">
-		<type>transmission_interface/SimpleTransmission</type>
-		<joint name="joint_1">
-			<hardwareInterface>hardware_interface/PositionJointInterface</hardwareInterface>
-		</joint>
-		<actuator name="motor_1">
-			<hardwareInterface>hardware_interface/PositionJointInterface</hardwareInterface>
-			<mechanicalReduction>1</mechanicalReduction>
-		</actuator>
-	</transmission>
 	<link name="J2">
 		<visual>
@@ -115,14 +105,4 @@
 		<dynamics damping="${joint_damping}" friction="${joint_friction}"/>
 	</joint>
-	<transmission name="trans_2">
-		<type>transmission_interface/SimpleTransmission</type>
-		<joint name="joint_2">
-			<hardwareInterface>hardware_interface/PositionJointInterface</hardwareInterface>
-		</joint>
-		<actuator name="motor_2">
-			<hardwareInterface>hardware_interface/PositionJointInterface</hardwareInterface>
-			<mechanicalReduction>1</mechanicalReduction>
-		</actuator>
-	</transmission>
 	<link name="J3">
 		<visual>
@@ -150,14 +130,4 @@
 		<dynamics damping="${joint_damping}" friction="${joint_friction}"/>
 	</joint>
-	<transmission name="trans_3">
-		<type>transmission_interface/SimpleTransmission</type>
-		<joint name="joint_3">
-			<hardwareInterface>hardware_interface/PositionJointInterface</hardwareInterface>
-		</joint>
-		<actuator name="motor_3">
-			<hardwareInterface>hardware_interface/PositionJointInterface</hardwareInterface>
-			<mechanicalReduction>1</mechanicalReduction>
-		</actuator>
-	</transmission>
 	<link name="J4">
 		<visual>
@@ -185,14 +155,4 @@
 		<dynamics damping="${joint_damping}" friction="${joint_friction}"/>
 	</joint>
-	<transmission name="trans_4">
-		<type>transmission_interface/SimpleTransmission</type>
-		<joint name="joint_4">
-			<hardwareInterface>hardware_interface/PositionJointInterface</hardwareInterface>
-		</joint>
-		<actuator name="motor_4">
-			<hardwareInterface>hardware_interface/PositionJointInterface</hardwareInterface>
-			<mechanicalReduction>1</mechanicalReduction>
-		</actuator>
-	</transmission>
 	<link name="J5">
 		<visual>
@@ -220,14 +180,4 @@
 		<dynamics damping="${joint_damping}" friction="${joint_friction}"/>
 	</joint>
-	<transmission name="trans_5">
-		<type>transmission_interface/SimpleTransmission</type>
-		<joint name="joint_5">
-			<hardwareInterface>hardware_interface/PositionJointInterface</hardwareInterface>
-		</joint>
-		<actuator name="motor_5">
-			<hardwareInterface>hardware_interface/PositionJointInterface</hardwareInterface>
-			<mechanicalReduction>1</mechanicalReduction>
-		</actuator>
-	</transmission>
 	<link name="J6">
 		<visual>
@@ -255,14 +205,4 @@
 		<dynamics damping="${joint_damping}" friction="${joint_friction}"/>
 	</joint>
-	<transmission name="trans_6">
-		<type>transmission_interface/SimpleTransmission</type>
-		<joint name="joint_6">
-			<hardwareInterface>hardware_interface/PositionJointInterface</hardwareInterface>
-		</joint>
-		<actuator name="motor_6">
-			<hardwareInterface>hardware_interface/PositionJointInterface</hardwareInterface>
-			<mechanicalReduction>1</mechanicalReduction>
-		</actuator>
-	</transmission>
 	<xacro:if value="${gripper_type != 'none'}">
 		<xacro:include filename="$(find denso_cobotta_description)/urdf/${gripper_type}.urdf.xacro" />

File: ROS2_ws/src/denso_cobotta_description/urdf/parallel.urdf.xacro (robot description, xacro)
@@ -20,4 +20,10 @@
 		</inertial>
 	</link>
+	<link name="gripper_tip"/>
+	<joint name="joint_tip" type="fixed">
+		<parent link="gripper_base"/>
+		<child link="gripper_tip"/>
+		<origin rpy="0.000000 0.000000 0.000000" xyz="0.000000 0.000000 0.065000"/>
+	</joint>
 	<joint name="joint_gripper_base" type="fixed">
 		<parent link="J6"/>
@@ -52,14 +58,4 @@
 		<dynamics damping="0" friction="0"/>
 	</joint>
-	<transmission name="trans_gripper">
-		<type>transmission_interface/SimpleTransmission</type>
-		<joint name="joint_gripper">
-			<hardwareInterface>hardware_interface/PositionJointInterface</hardwareInterface>
-		</joint>
-		<actuator name="motor_gripper">
-			<hardwareInterface>hardware_interface/PositionJointInterface</hardwareInterface>
-			<mechanicalReduction>1</mechanicalReduction>
-		</actuator>
-	</transmission>
 	<link name="right_finger">
 		<visual>

Commit message: changed urdf scale parameters and removed innertia values

File: ROS2_ws/src/denso_cobotta_description/urdf/cobotta.urdf.xacro (robot description, xacro)
@@ -3,34 +3,5 @@
 	<xacro:arg name="gripper_type" default="parallel"/>
 	<xacro:property name="gripper_type" value="$(arg gripper_type)" />
-	<!-- Parameters for gazebo simulation.
-		NOTE: These are roughly estimated values.
-	-->
-	<xacro:property name="joint_damping" value="0.001" />
-	<xacro:property name="joint_friction" value="0.61" />
-	<xacro:property name="base_mass" value="1.4" />
-	<xacro:property name="J1_mass" value="1.29" />
-	<xacro:property name="J2_mass" value="0.39" />
-	<xacro:property name="J3_mass" value="0.35" />
-	<xacro:property name="J4_mass" value="0.35" />
-	<xacro:property name="J5_mass" value="0.19" />
-	<xacro:property name="J6_mass" value="0.03" />
-	<!-- Macro for calculating inertial matrix-->
-	<xacro:macro name="inertia_macro" params="radius height mass *origin">
-    	<inertial>
-    	  <mass value="${mass}" />
-		  <xacro:insert_block name="origin" />
-    	  <inertia ixx="${((1 / 4) * mass * radius * radius) + ((1 / 12) * mass * height * height)}" ixy="0.0" ixz="0.0"
-    	    iyy="${((1 / 4) * mass * radius * radius) + ((1 / 12) * mass * height * height)}" iyz="0.0"
-    	    izz="${(1 / 2) * mass * radius * radius}" />
-    	</inertial>
-  	</xacro:macro>
-	<!-- plugin for Gazebo -->
-	<gazebo>
-		<plugin name="gazebo_ros_control" filename="libgazebo_ros_control.so">
-			<robotNamespace>/cobotta</robotNamespace>
-      <robotSimType>gazebo_ros_control/DefaultRobotHWSim</robotSimType>
-      <legacyModeNS>true</legacyModeNS>
-		</plugin>
-	</gazebo>
+	<xacro:property name="scale_value" value="100.0"/>
 	<link name="world"/>
 	<joint name="joint_w" type="fixed">
@@ -42,5 +13,5 @@
 			<origin rpy="0 0 0" xyz="0 0 0"/>
 			<geometry>
-				<mesh filename="package://denso_cobotta_description/meshes/visual/robot/base_link.dae" scale="1 1 1"/>
+				<mesh filename="package://denso_cobotta_description/meshes/visual/robot/base_link.dae" scale="${scale_value} ${scale_value} ${scale_value}"/>
 			</geometry>
 		</visual>
@@ -48,16 +19,13 @@
 			<origin rpy="0 0 0" xyz="0 0 0"/>
 			<geometry>
-				<mesh filename="package://denso_cobotta_description/meshes/collision/robot/base_link.dae" scale="1 1 1"/>
+				<mesh filename="package://denso_cobotta_description/meshes/collision/robot/base_link.dae" scale="${scale_value} ${scale_value} ${scale_value}"/>
 			</geometry>
 		</collision>
-		<xacro:inertia_macro radius="0.08" height="0.06" mass="${base_mass}">
-			<origin rpy="0.000000 0.000000 0.000000" xyz="-0.021310 0.000002 0.044011"/>
-		</xacro:inertia_macro>
 	</link>
-	<link name="J1">
+	<link name="link_1">
 		<visual>
 			<origin rpy="0 0 0" xyz="0 0 0"/>
 			<geometry>
-				<mesh filename="package://denso_cobotta_description/meshes/visual/robot/J1.dae" scale="1 1 1"/>
+				<mesh filename="package://denso_cobotta_description/meshes/visual/robot/link_1.dae" scale="${scale_value} ${scale_value} ${scale_value}"/>
 			</geometry>
 		</visual>
@@ -65,24 +33,20 @@
 			<origin rpy="0 0 0" xyz="0 0 0"/>
 			<geometry>
-				<mesh filename="package://denso_cobotta_description/meshes/collision/robot/J1.dae" scale="1 1 1"/>
+				<mesh filename="package://denso_cobotta_description/meshes/collision/robot/link_1.dae" scale="${scale_value} ${scale_value} ${scale_value}"/>
 			</geometry>
 		</collision>
-		<xacro:inertia_macro radius="0.06" height="0.1" mass="${J1_mass}">
-			<origin rpy="0.000000 0.000000 0.000000" xyz="0.000000 0.000000 0.15" />
-		</xacro:inertia_macro>
 	</link>
 	<joint name="joint_1" type="revolute">
 		<parent link="base_link"/>
-		<child link="J1" />
+		<child link="link_1" />
 		<origin rpy="0.000000 0.000000 0.000000" xyz="0.000000 0.000000 0.000000" />
 		<axis xyz="-0.000000 -0.000000 1.000000" />
-		<limit effort="10" lower="-2.617994" upper="2.617994" velocity="0.40317105721069" />
-		<dynamics damping="${joint_damping}" friction="${joint_friction}" />
+		<limit effort="${scale_value * 10000}" lower="-2.617994" upper="2.617994" velocity="${scale_value * 0.403171057210690}" />
 	</joint>
-	<link name="J2">
+	<link name="link_2">
 		<visual>
 			<origin rpy="0 0 0" xyz="0 0 0"/>
 			<geometry>
-				<mesh filename="package://denso_cobotta_description/meshes/visual/robot/J2.dae" scale="1 1 1"/>
+				<mesh filename="package://denso_cobotta_description/meshes/visual/robot/link_2.dae" scale="${scale_value} ${scale_value} ${scale_value}"/>
 			</geometry>
 		</visual>
@@ -90,24 +54,20 @@
 			<origin rpy="0 0 0" xyz="0 0 0"/>
 			<geometry>
-				<mesh filename="package://denso_cobotta_description/meshes/collision/robot/J2.dae" scale="1 1 1"/>
+				<mesh filename="package://denso_cobotta_description/meshes/collision/robot/link_2.dae" scale="${scale_value} ${scale_value} ${scale_value}"/>
 			</geometry>
 		</collision>
-		<xacro:inertia_macro radius="0.03" height="0.12" mass="${J2_mass}">
-			<origin rpy="0.000000 0.000000 0.000000" xyz="-0.020000 0.100000 0.070000" />
-		</xacro:inertia_macro>
 	</link>
 	<joint name="joint_2" type="revolute">
-		<parent link="J1"/>
-		<child link="J2"/>
-		<origin rpy="0.000000 0.000000 0.000000" xyz="0.000000 0.000000 0.180000" />
+		<parent link="link_1"/>
+		<child link="link_2"/>
+		<origin rpy="0.000000 0.000000 0.000000" xyz="0.000000 0.000000 ${scale_value * 0.180000}" />
 		<axis xyz="-0.000000 1.000000 -0.000000" />
-		<limit effort="10" lower="-1.047198" upper="1.745329" velocity="0.392175482923126" />
-		<dynamics damping="${joint_damping}" friction="${joint_friction}"/>
+		<limit effort="${scale_value * 10000}" lower="-1.047198" upper="1.745329" velocity="${scale_value * 0.392175482923126}" />
 	</joint>
-	<link name="J3">
+	<link name="link_3">
 		<visual>
 			<origin rpy="0 0 0" xyz="0 0 0"/>
 			<geometry>
-				<mesh filename="package://denso_cobotta_description/meshes/visual/robot/J3.dae" scale="1 1 1"/>
+				<mesh filename="package://denso_cobotta_description/meshes/visual/robot/link_3.dae" scale="${scale_value} ${scale_value} ${scale_value}"/>
 			</geometry>
 		</visual>
@@ -115,24 +75,20 @@
 			<origin rpy="0 0 0" xyz="0 0 0"/>
 			<geometry>
-				<mesh filename="package://denso_cobotta_description/meshes/collision/robot/J3.dae" scale="1 1 1"/>
+				<mesh filename="package://denso_cobotta_description/meshes/collision/robot/link_3.dae" scale="${scale_value} ${scale_value} ${scale_value}"/>
 			</geometry>
 		</collision>
-		<xacro:inertia_macro radius="0.03" height="0.11" mass="${J3_mass}">
-			<origin rpy="0.000000 0.000000 0.000000" xyz="-0.01000 0.020000 0.030000" />
-		</xacro:inertia_macro>
 	</link>
 	<joint name="joint_3" type="revolute">
-		<parent link="J2"/>
-		<child link="J3"/>
-		<origin rpy="0.000000 0.000000 0.000000" xyz="0.000000 0.000000 0.165000" />
+		<parent link="link_2"/>
+		<child link="link_3"/>
+		<origin rpy="0.000000 0.000000 0.000000" xyz="0.000000 0.000000 ${scale_value * 0.165000}" />
 		<axis xyz="-0.000000 1.000000 -0.000000" />
-		<limit effort="10" lower="0.3141593" upper="2.443461" velocity="0.725707902979242" />
-		<dynamics damping="${joint_damping}" friction="${joint_friction}"/>
+		<limit effort="${scale_value * 10000}" lower="0.3141593" upper="2.443461" velocity="${scale_value * 0.725707902979242}" />
 	</joint>
-	<link name="J4">
+	<link name="link_4">
 		<visual>
 			<origin rpy="0 0 0" xyz="0 0 0"/>
 			<geometry>
-				<mesh filename="package://denso_cobotta_description/meshes/visual/robot/J4.dae" scale="1 1 1"/>
+				<mesh filename="package://denso_cobotta_description/meshes/visual/robot/link_4.dae" scale="${scale_value} ${scale_value} ${scale_value}"/>
 			</geometry>
 		</visual>
@@ -140,24 +96,20 @@
 			<origin rpy="0 0 0" xyz="0 0 0"/>
 			<geometry>
-				<mesh filename="package://denso_cobotta_description/meshes/collision/robot/J4.dae" scale="1 1 1"/>
+				<mesh filename="package://denso_cobotta_description/meshes/collision/robot/link_4.dae" scale="${scale_value} ${scale_value} ${scale_value}"/>
 			</geometry>
 		</collision>
-		<xacro:inertia_macro radius="0.03" height="0.11" mass="${J4_mass}">
-			<origin rpy="0.000000 0.000000 0.000000" xyz="0.0000 0.000000 0.055000"/>
-		</xacro:inertia_macro>
 	</link>
 	<joint name="joint_4" type="revolute">
-		<parent link="J3"/>
-		<child link="J4"/>
-		<origin rpy="0.000000 0.000000 0.000000" xyz="-0.012000 0.020000 0.088000" />
+		<parent link="link_3"/>
+		<child link="link_4"/>
+		<origin rpy="0.000000 0.000000 0.000000" xyz="${scale_value * (-0.012000)} ${scale_value * 0.020000} ${scale_value * 0.088000}" />
 		<axis xyz="-0.000000 -0.000000 1.000000" />
-		<limit effort="10" lower="-2.96706" upper="2.96706" velocity="0.739146938219599" />
-		<dynamics damping="${joint_damping}" friction="${joint_friction}"/>
+		<limit effort="${scale_value * 10000}" lower="-2.96706" upper="2.96706" velocity="${scale_value * 0.739146938219599}" />
 	</joint>
-	<link name="J5">
+	<link name="link_5">
 		<visual>
 			<origin rpy="0 0 0" xyz="0 0 0"/>
 			<geometry>
-				<mesh filename="package://denso_cobotta_description/meshes/visual/robot/J5.dae" scale="1 1 1"/>
+				<mesh filename="package://denso_cobotta_description/meshes/visual/robot/link_5.dae" scale="${scale_value} ${scale_value} ${scale_value}"/>
 			</geometry>
 		</visual>
@@ -165,24 +117,20 @@
 			<origin rpy="0 0 0" xyz="0 0 0"/>
 			<geometry>
-				<mesh filename="package://denso_cobotta_description/meshes/collision/robot/J5.dae" scale="1 1 1"/>
+				<mesh filename="package://denso_cobotta_description/meshes/collision/robot/link_5.dae" scale="${scale_value} ${scale_value} ${scale_value}"/>
 			</geometry>
 		</collision>
-		<xacro:inertia_macro radius="0.03" height="0.06" mass="${J5_mass}">
-			<origin rpy="0.000000 0.000000 0.000000" xyz="0.000000 -0.040000 0.015000"/>
-		</xacro:inertia_macro>
 	</link>
 	<joint name="joint_5" type="revolute">
-		<parent link="J4"/>
-		<child link="J5"/>
-		<origin rpy="0.000000 0.000000 0.000000" xyz="0.000000 -0.020000 0.089500" />
+		<parent link="link_4"/>
+		<child link="link_5"/>
+		<origin rpy="0.000000 0.000000 0.000000" xyz="0.000000 ${scale_value * (-0.020000)} ${scale_value * 0.089500}" />
 		<axis xyz="-0.000000 1.000000 -0.000000" />
-		<limit effort="10" lower="-1.658063" upper="2.356194" velocity="0.739146938219599" />
-		<dynamics damping="${joint_damping}" friction="${joint_friction}"/>
+		<limit effort="${scale_value * 10000}" lower="-1.658063" upper="2.356194" velocity="${scale_value * 0.739146938219599}" />
 	</joint>
-	<link name="J6">
+	<link name="link_6">
 		<visual>
 			<origin rpy="0 0 0" xyz="0 0 0"/>
 			<geometry>
-				<mesh filename="package://denso_cobotta_description/meshes/visual/robot/J6.dae" scale="1 1 1"/>
+				<mesh filename="package://denso_cobotta_description/meshes/visual/robot/link_6.dae" scale="${scale_value} ${scale_value} ${scale_value}"/>
 			</geometry>
 		</visual>
@@ -190,18 +138,14 @@
 			<origin rpy="0 0 0" xyz="0 0 0"/>
 			<geometry>
-				<mesh filename="package://denso_cobotta_description/meshes/collision/robot/J6.dae" scale="1 1 1"/>
+				<mesh filename="package://denso_cobotta_description/meshes/collision/robot/link_6.dae" scale="${scale_value} ${scale_value} ${scale_value}"/>
 			</geometry>
 		</collision>
-		<xacro:inertia_macro radius="0.03" height="0.01" mass="${J6_mass}">
-			<origin rpy="0.000000 0.000000 0.000000" xyz="0.000000 0.000000 0.000000" />
-		</xacro:inertia_macro>
 	</link>
 	<joint name="joint_6" type="revolute">
-		<parent link="J5"/>
-		<child link="J6"/>
-		<origin rpy="0.000000 0.000000 0.000000" xyz="0.000000 -0.044500 0.042000" />
+		<parent link="link_5"/>
+		<child link="link_6"/>
+		<origin rpy="0.000000 0.000000 0.000000" xyz="0.000000 ${scale_value * (-0.044500)} ${scale_value * 0.042000}" />
 		<axis xyz="-0.000000 -0.000000 1.000000" />
-		<limit effort="10" lower="-2.96706" upper="2.96706" velocity="1.1093312725676" />
-		<dynamics damping="${joint_damping}" friction="${joint_friction}"/>
+		<limit effort="${scale_value * 10000}" lower="-2.96706" upper="2.96706" velocity="${scale_value * 1.109331272567600}" />
 	</joint>
 	<xacro:if value="${gripper_type != 'none'}">

File: ROS2_ws/src/denso_cobotta_description/urdf/parallel.urdf.xacro (robot description, xacro)
@@ -5,5 +5,5 @@
 			<origin rpy="0 0 0" xyz="0.000000 0.000000 0.000000"/>
 			<geometry>
-				<mesh filename="package://denso_cobotta_description/meshes/visual/tool/gripper_base.dae" scale="1 1 1"/>
+				<mesh filename="package://denso_cobotta_description/meshes/visual/tool/gripper_base.dae" scale="${scale_value} ${scale_value} ${scale_value}"/>
 			</geometry>
 		</visual>
@@ -11,5 +11,5 @@
 			<origin rpy="0 0 0" xyz="0 0 0"/>
 			<geometry>
-				<mesh filename="package://denso_cobotta_description/meshes/collision/tool/gripper_base.dae" scale="1 1 1"/>
+				<mesh filename="package://denso_cobotta_description/meshes/collision/tool/gripper_base.dae" scale="${scale_value} ${scale_value} ${scale_value}"/>
 			</geometry>
 		</collision>
@@ -24,8 +24,8 @@
 		<parent link="gripper_base"/>
 		<child link="gripper_tip"/>
-		<origin rpy="0.000000 0.000000 0.000000" xyz="0.000000 0.000000 0.065000"/>
+		<origin rpy="0.000000 0.000000 0.000000" xyz="0.000000 0.000000 ${scale_value * 0.06500}"/>
 	</joint>
 	<joint name="joint_gripper_base" type="fixed">
-		<parent link="J6"/>
+		<parent link="link_6"/>
 		<child link="gripper_base"/>
 		<origin rpy="0.000000 0.000000 0.000000" xyz="0.000000 0.000000 0.0000000"/>
@@ -33,13 +33,13 @@
 	<link name="left_finger">
 		<visual>
-			<origin rpy="0.000000 0.000000 0.000000" xyz="0.000000 0.000000 -0.060000"/>
+			<origin rpy="0.000000 0.000000 0.000000" xyz="0.000000 0.000000 ${scale_value * (-0.060000)}"/>
 			<geometry>
-				<mesh filename="package://denso_cobotta_description/meshes/visual/tool/left_finger.dae" scale="1 1 1"/>
+				<mesh filename="package://denso_cobotta_description/meshes/visual/tool/left_finger.dae" scale="${scale_value} ${scale_value} ${scale_value}"/>
 			</geometry>
 		</visual>
 		<collision>
-			<origin rpy="0 0 0" xyz="0.000000 0.000000 -0.060000"/>
+			<origin rpy="0 0 0" xyz="0.000000 0.000000 ${scale_value * (-0.060000)}"/>
 			<geometry>
-				<mesh filename="package://denso_cobotta_description/meshes/collision/tool/left_finger.dae" scale="1 1 1"/>
+				<mesh filename="package://denso_cobotta_description/meshes/collision/tool/left_finger.dae" scale="${scale_value} ${scale_value} ${scale_value}"/>
 			</geometry>
 		</collision>
@@ -53,20 +53,20 @@
 		<parent link="gripper_base"/>
 		<child link="left_finger"/>
-		<origin rpy="0.000000 0.000000 0.000000" xyz="0.000000 0.000000 0.06000"/>
+		<origin rpy="0.000000 0.000000 0.000000" xyz="0.000000 0.000000 ${scale_value * 0.060000}"/>
 		<axis xyz="-0.000000 1.000000 -0.000000"/>
-		<limit effort="20" lower="0.000000" upper="0.015000" velocity="0.040000"/>
+		<limit effort="${scale_value * 200000}" lower="0.000000" upper="${scale_value * 0.0150000}" velocity="${scale_value * 18.000000}"/>
 		<dynamics damping="0" friction="0"/>
 	</joint>
 	<link name="right_finger">
 		<visual>
-			<origin rpy="0.000000 0.000000 0.000000" xyz="0.000000 0.000000 -0.060000"/>
+			<origin rpy="0.000000 0.000000 0.000000" xyz="0.000000 0.000000 ${scale_value * (-0.060000)}"/>
 			<geometry>
-				<mesh filename="package://denso_cobotta_description/meshes/visual/tool/right_finger.dae" scale="1 1 1"/>
+				<mesh filename="package://denso_cobotta_description/meshes/visual/tool/right_finger.dae" scale="${scale_value} ${scale_value} ${scale_value}"/>
 			</geometry>
 		</visual>
 		<collision>
-			<origin rpy="0 0 0" xyz="0.000000 0.000000 -0.060000"/>
+			<origin rpy="0 0 0" xyz="0.000000 0.000000 ${scale_value * (-0.060000)}"/>
 			<geometry>
-				<mesh filename="package://denso_cobotta_description/meshes/collision/tool/right_finger.dae" scale="1 1 1"/>
+				<mesh filename="package://denso_cobotta_description/meshes/collision/tool/right_finger.dae" scale="${scale_value} ${scale_value} ${scale_value}"/>
 			</geometry>
 		</collision>
@@ -81,7 +81,7 @@
 		<child link="right_finger"/>
 		<mimic joint="joint_gripper" multiplier="-1.000000" offset="0.000000"/>
-		<origin rpy="0.000000 0.000000 0.000000" xyz="0.000000 0.000000 0.060000"/>
+		<origin rpy="0.000000 0.000000 0.000000" xyz="0.000000 0.000000 ${scale_value * (0.060000)}"/>
 		<axis xyz="-0.000000 1.000000 -0.000000"/>
-		<limit effort="20" lower="-0.015000" upper="0.000000" velocity="0.040000"/>
+		<limit effort="${scale_value * 200000}" lower="${scale_value * (-0.0150000)}" upper="0.000000" velocity="${scale_value * 18.00000}"/>
 		<dynamics damping="0" friction="0"/>
 	</joint>
