Commit message: Denso Wave cobotta files changes to make it more standarlized

File: ROS2_ws/src/denso_cobotta_description/urdf/denso_cobotta.urdf.xacro (robot description, xacro)
@@ -1,4 +1,4 @@
 <?xml version="1.0" encoding="UTF-8"?>
-<robot name="cobotta" xmlns:xacro="http://www.ros.org/wiki/xacro">
+<robot name="denso_cobotta" xmlns:xacro="http://www.ros.org/wiki/xacro">
 	<xacro:arg name="gripper_type" default="parallel"/>
 	<xacro:property name="gripper_type" value="$(arg gripper_type)" />

File: ROS2_ws/src/denso_cobotta_description/urdf/parallel.urdf.xacro (robot description, xacro)
@@ -1,4 +1,4 @@
 <?xml version="1.0" encoding="UTF-8"?>
-<robot name="cobotta" xmlns:xacro="http://www.ros.org/wiki/xacro">
+<robot name="denso_cobotta" xmlns:xacro="http://www.ros.org/wiki/xacro">
 	<link name="gripper_base">
 		<visual>

File: ROS2_ws/src/denso_cobotta_moveit_config/config/denso_cobotta.ros2_control.xacro (robot description, xacro)
@@ -1,5 +1,5 @@
 <?xml version="1.0"?>
 <robot xmlns:xacro="http://www.ros.org/wiki/xacro">
-    <xacro:macro name="cobotta_ros2_control" params="name initial_positions_file">
+    <xacro:macro name="denso_cobotta_ros2_control" params="name initial_positions_file">
         <xacro:property name="initial_positions" value="${xacro.load_yaml(initial_positions_file)['initial_positions']}"/>
         <ros2_control name="${name}" type="system">

Commit message: Changes to Cobotta and VP robots files

File: ROS2_ws/src/denso_cobotta_description/urdf/denso_cobotta.urdf.xacro (robot description, xacro)
@@ -1,5 +1,5 @@
 <?xml version="1.0" encoding="UTF-8"?>
 <robot name="denso_cobotta" xmlns:xacro="http://www.ros.org/wiki/xacro">
-	<xacro:arg name="gripper_type" default="parallel"/>
+	<xacro:arg name="gripper_type" default="taiyo"/>
 	<xacro:property name="gripper_type" value="$(arg gripper_type)" />
 	<xacro:property name="scale_value" value="100.0"/>
@@ -8,4 +8,5 @@
 		<parent link="world"/>
 		<child link="base_link"/>
+		<origin rpy="0.000000 0.000000 1.5707" xyz="17.00 -6.0 18.16" />
 	</joint>
 	<link name="base_link">

File: ROS2_ws/src/denso_vp6242_description/urdf/denso_vp6242.urdf.xacro (robot description, xacro)
@@ -1,5 +1,5 @@
 <?xml version="1.0" encoding="UTF-8"?>
 <robot name="denso_vp6242" xmlns:xacro="http://www.ros.org/wiki/xacro">
-	<xacro:arg name="gripper_type" default="tayo"/>
+	<xacro:arg name="gripper_type" default="taiyo"/>
 	<xacro:property name="gripper_type" value="$(arg gripper_type)" />
 	<xacro:property name="scale_value" value="100.0"/>
