Commit message: Added the vp6242 gripper to the URDF files

File: ROS2_ws/src/denso_vp6242_description/urdf/vp6242.urdf (robot description, URDF)
Before this commit: robot vp6242, 9 links, 8 joints
Links:
- added link gripper_body; collision box size=0.11 0.04 0.084; visual box size=0.11 0.04 0.084
- added link left_claw; collision box size=0.05075 0.015 0.0136; visual box size=0.05075 0.015 0.0136
- added link peak_tool
- added link right_claw; collision box size=0.05075 0.015 0.0136; visual box size=0.05075 0.015 0.0136
- added link robot_gripper_interface1; collision cylinder length=0.009 radius=0.04; visual cylinder length=0.009 radius=0.04
- added link robot_gripper_interface2; collision cylinder length=0.009 radius=0.04; visual cylinder length=0.009 radius=0.04
Joints:
- added joint interface_to_gripper_body: type fixed, parent robot_gripper_interface2, child gripper_body, origin xyz=0.0 0.0 0.009 rpy=0 0 0
- added joint left_claw_joint: type fixed, parent gripper_body, child left_claw, origin xyz=-0.029625 0 0.084 rpy=0 0 0
- added joint peak_tool: type fixed, parent gripper_body, child peak_tool, origin xyz=0 0 0.0976 rpy=0 3.14159265359 0
- added joint right_claw_joint: type fixed, parent gripper_body, child right_claw, origin xyz=0.029625 0 0.084 rpy=0 0 0
- added joint robot_to_gripper: type fixed, parent tool0, child robot_gripper_interface1, origin xyz=0 0 0 rpy=0 0 1.57079632679
- added joint robot_to_gripper_interface_2: type fixed, parent robot_gripper_interface1, child robot_gripper_interface2, origin xyz=0 0 0.009 rpy=0 0 0

Commit message: vp6242 robot package

File: ROS2_ws/src/denso_vp6242_description/urdf/vp6242.urdf (robot description, URDF)
Before this commit: robot vp6242, 15 links, 14 joints
Links:
- link base_link: geometry collision mesh filename=package://denso_vp6242_description/meshes/collision/base.dae scale=${scale_value * 0.001} ${scale_value * 0.001} ${scale_value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; visual mesh filename=package://denso_vp6242_description/meshes/visual/base.dae scale=${scale_value * 0.001} ${scale_value * 0.001} ${scale_value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
- link gripper_body: geometry collision box size=${scale_value*0.11} ${scale_value*0.04} ${scale_value*0.084}; visual box size=${scale_value*0.11} ${scale_value*0.04} ${scale_value*0.084}
- link left_claw: geometry collision box size=${scale_value*0.05075} ${scale_value*0.015} ${scale_value*0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; visual box size=${scale_value*0.05075} ${scale_value*0.015} ${scale_value*0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
- link link1: geometry collision mesh filename=package://denso_vp6242_description/meshes/collision/link1.d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 scale=${scale_value * 0.001} ${scale_value * 0.001} ${scale_value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; visual mesh filename=package://denso_vp6242_description/meshes/visual/link1.dae scale=${scale_value * 0.001} ${scale_value * 0.001} ${scale_value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
- link link2: geometry collision mesh filename=package://denso_vp6242_description/meshes/collision/link2.d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 scale=${scale_value * 0.001} ${scale_value * 0.001} ${scale_value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; visual mesh filename=package://denso_vp6242_description/meshes/visual/link2.dae scale=${scale_value * 0.001} ${scale_value * 0.001} ${scale_value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
- link link3: geometry collision mesh filename=package://denso_vp6242_description/meshes/collision/link3.d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 scale=${scale_value * 0.001} ${scale_value * 0.001} ${scale_value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; visual mesh filename=package://denso_vp6242_description/meshes/visual/link3.dae scale=${scale_value * 0.001} ${scale_value * 0.001} ${scale_value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
- link link4: geometry collision mesh filename=package://denso_vp6242_description/meshes/collision/link4.d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 scale=${scale_value * 0.001} ${scale_value * 0.001} ${scale_value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; visual mesh filename=package://denso_vp6242_description/meshes/visual/link4.dae scale=${scale_value * 0.001} ${scale_value * 0.001} ${scale_value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
- link link5: geometry collision mesh filename=package://denso_vp6242_description/meshes/collision/link5.d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 scale=${scale_value * 0.001} ${scale_value * 0.001} ${scale_value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; visual mesh filename=package://denso_vp6242_description/meshes/visual/link5.dae scale=${scale_value * 0.001} ${scale_value * 0.001} ${scale_value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
- link link6: geometry collision cylinder length=${scale_value*0.01} radius=${scale_value*0.0205}; visual cylinder length=${scale_value*0.01} radius=${scale_value*0.0205}
- link right_claw: geometry collision box size=${scale_value*0.05075} ${scale_value*0.015} ${scale_value*0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; visual box size=${scale_value*0.05075} ${scale_value*0.015} ${scale_value*0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
- link robot_gripper_interface1: geometry collision cylinder length=${scale_value*0.009} radius=${scale_value*0.04}; visual cylinder length=${scale_value*0.009} radius=${scale_value*0.04}
- link robot_gripper_interface2: geometry collision cylinder length=${scale_value*0.009} radius=${scale_value*0.04}; visual cylinder length=${scale_value*0.009} radius=${scale_value*0.04}
Joints:
- joint interface_to_gripper_body: origin xyz=0.0 0.0 0.009 rpy=0 0 0 -> xyz=0.0 0.0 ${scale_value*0.009} rpy=0 0 0
- joint joint1: origin xyz=0.0 0.0 0.155 rpy=0 0 0 -> xyz=0.0 0.0 ${scale_value*0.155} rpy=0 0 0
- joint joint2: origin xyz=0.0 0.0 0.125 rpy=0 0 0 -> xyz=0.0 0.0 ${scale_value*0.125} rpy=0 0 0
- joint joint3: origin xyz=0.0 0.0 0.210 rpy=0 0 0 -> xyz=0.0 0.0 ${scale_value*0.210} rpy=0 0 0
- joint joint4: origin xyz=-0.075 0.0 0.0 rpy=0 0 0 -> xyz=${-scale_value*0.075} 0.0 0.0 rpy=0 0 0
- joint joint5: origin xyz=0.0 0.0 0.210 rpy=0 0 0 -> xyz=0.0 0.0 ${scale_value*0.210} rpy=0 0 0
- joint joint6: origin xyz=0.0 0.0 0.07 rpy=0 0 0 -> xyz=0.0 0.0 ${scale_value*0.07} rpy=0 0 0
- joint left_claw_joint: origin xyz=-0.029625 0 0.084 rpy=0 0 0 -> xyz=${-scale_value*0.029625} 0 ${scale_value*0.084} rpy=0 0 0
- joint peak_tool: origin xyz=0 0 0.0976 rpy=0 3.14159265359 0 -> xyz=0 0 ${scale_value*0.0976} rpy=0 3.14159265359 0
- joint right_claw_joint: origin xyz=0.029625 0 0.084 rpy=0 0 0 -> xyz=${scale_value*0.029625} 0 ${scale_value*0.084} rpy=0 0 0
- joint robot_to_gripper_interface_2: origin xyz=0 0 0.009 rpy=0 0 0 -> xyz=0 0 ${scale_value*0.009} rpy=0 0 0
