Commit message: VP6242 robot is correctly performing assembly. The path execution problem was solved

File: ROS2_ws/src/denso_vp6242_description/urdf/vp6242.urdf.xacro (robot description, xacro)
@@ -156,5 +156,5 @@
 		<child link="tool0"/>
 		<origin rpy="0 0 0" xyz="0 0 0"/>
-	</joint>
+  	</joint>
 	<link name="robot_gripper_interface1">
 		<collision>
@@ -261,17 +261,24 @@
 	</joint>
 	<!--joint of gripper and claw-->
-	<joint name="right_claw_joint" type="fixed">
+	<joint name="right_claw_joint" type="prismatic">
 		<parent link="gripper_body"/>
 		<child link="right_claw"/>
-		<origin rpy="0 0 0" xyz="${scale_value*0.029625} 0 ${scale_value*0.084}"/>
-	</joint>
-	<joint name="left_claw_joint" type="fixed">
+		<origin rpy="0.000000 0.000000 0.000000" xyz="${scale_value*0.029625} 0 ${scale_value*0.084}"/>
+		<axis xyz="1.000000 0.000000 -0.000000"/>
+		<limit effort="${scale_value * 200000}" lower="-${scale_value * 0.0015000}" upper="0.0" velocity="0.1"/>
+		<dynamics damping="0" friction="0"/>
+	</joint>
+	<joint name="left_claw_joint" type="prismatic">
 		<parent link="gripper_body"/>
 		<child link="left_claw"/>
-		<origin rpy="0 0 0" xyz="${scale_value*(-0.029625)} 0 ${scale_value*0.084}"/>
+		<mimic joint="right_claw_joint" multiplier="-1.000000" offset="0.000000"/>
+		<origin rpy="0.000000 0.000000 0.000000" xyz="${scale_value*(-0.029625)} 0 ${scale_value*0.084}"/>
+		<axis xyz="1.000000 0.000000 -0.000000"/>
+		<limit effort="${scale_value * 200000}" lower="0.0" upper="${scale_value * (0.00150000)}" velocity="0.1"/>
+		<dynamics damping="0" friction="0"/>
 	</joint>
 	<!--joint of gripper and peak tool-->
 	<joint name="peak_tool" type="fixed">
-		<origin rpy="0 .14159265359 0" xyz="0 0 ${scale_value*0.0976}"/>
+		<origin rpy="0 3.14159265359 0" xyz="0 0 ${scale_value*0.0976}"/>
 		<parent link="gripper_body"/>
 		<child link="peak_tool"/>

File: ROS2_ws/src/denso_vp6242_moveit_config/config/vp6242.ros2_control.xacro (robot description, xacro)
@@ -50,4 +50,11 @@
                 <state_interface name="velocity"/>
             </joint>
+            <joint name="right_claw_joint">
+                <command_interface name="position"/>
+                <state_interface name="position">
+                  <param name="initial_value">${initial_positions['right_claw_joint']}</param>
+                </state_interface>
+                <state_interface name="velocity"/>
+            </joint>
         </ros2_control>
     </xacro:macro>

File: ROS2_ws/src/denso_vp6242_moveit_config/config/vp6242.urdf.xacro (robot description, xacro)
@@ -3,5 +3,5 @@
     <xacro:arg name="initial_positions_file" default="initial_positions.yaml" />
     <!-- Import vp6242 urdf file -->
-    <xacro:include filename="$(find denso_vp6242_description)/urdf/vp6242.urdf" />
+    <xacro:include filename="$(find denso_vp6242_description)/urdf/vp6242.urdf.xacro" />
     <!-- Import control_xacro -->
     <xacro:include filename="vp6242.ros2_control.xacro" />
