Commit message: changes to denso vp6242 naming convention to work with the new robot spawning method

File: ROS2_ws/src/denso_vp6242_description/urdf/denso_vp6242.urdf.xacro (robot description, xacro)
@@ -1,4 +1,4 @@
 <?xml version="1.0" encoding="UTF-8"?>
-<robot name="vp6242" xmlns:xacro="http://www.ros.org/wiki/xacro">
+<robot name="denso_vp6242" xmlns:xacro="http://www.ros.org/wiki/xacro">
 	<xacro:property name="scale_value" value="100.0"/>
 	<link name="world"/>

File: ROS2_ws/src/denso_vp6242_moveit_config/config/denso_vp6242.ros2_control.xacro (robot description, xacro)
@@ -1,5 +1,5 @@
 <?xml version="1.0"?>
 <robot xmlns:xacro="http://www.ros.org/wiki/xacro">
-    <xacro:macro name="vp6242_ros2_control" params="name initial_positions_file">
+    <xacro:macro name="denso_vp6242_ros2_control" params="name initial_positions_file">
         <xacro:property name="initial_positions" value="${xacro.load_yaml(initial_positions_file)['initial_positions']}"/>
         <ros2_control name="${name}" type="system">

Commit message: Denso Wave vp6242 files changes to make it more standarlized

File: ROS2_ws/src/denso_vp6242_description/urdf/denso_vp6242.urdf.xacro (robot description, xacro)
@@ -1,4 +1,6 @@
 <?xml version="1.0" encoding="UTF-8"?>
 <robot name="denso_vp6242" xmlns:xacro="http://www.ros.org/wiki/xacro">
+	<xacro:arg name="gripper_type" default="tayo"/>
+	<xacro:property name="gripper_type" value="$(arg gripper_type)" />
 	<xacro:property name="scale_value" value="100.0"/>
 	<link name="world"/>
@@ -9,87 +11,122 @@
 	<link name="base_link">
 		<visual>
+			<origin rpy="-1.570796 3.141592 0" xyz="0 0 0"/>
 			<geometry>
-				<mesh filename="package://denso_vp6242_description/meshes/visual/base.dae" scale="${scale_value * 0.001} ${scale_value * 0.001} ${scale_value * 0.001}"/>
+				<mesh filename="package://denso_vp6242_description/meshes/visual/robot/base_link.dae" scale="${scale_value} ${scale_value} ${scale_value}"/>
 			</geometry>
-			<origin rpy="-1.570796 3.141592 0" xyz="0 0 0"/>
 		</visual>
 		<collision>
+			<origin rpy="-1.570796 3.141592 0" xyz="0 0 0"/>
 			<geometry>
-				<mesh filename="package://denso_vp6242_description/meshes/collision/base.dae" scale="${scale_value*0.001} ${scale_value*0.001} ${scale_value*0.001}"/>
+				<mesh filename="package://denso_vp6242_description/meshes/collision/robot/base_link.dae" scale="${scale_value} ${scale_value} ${scale_value}"/>
 			</geometry>
-			<origin rpy="-1.570796 3.141592 0" xyz="0 0 0"/>
 		</collision>
 	</link>
-	<link name="link1">
+	<link name="link_1">
 		<visual>
+			<origin rpy="-1.570796 3.141592 0" xyz="0 0 0"/>
 			<geometry>
-				<mesh filename="package://denso_vp6242_description/meshes/visual/link1.dae" scale="${scale_value*0.001} ${scale_value*0.001} ${scale_value*0.001}"/>
+				<mesh filename="package://denso_vp6242_description/meshes/visual/robot/link_1.dae" scale="${scale_value} ${scale_value} ${scale_value}"/>
 			</geometry>
-			<origin rpy="-1.570796 3.141592 0" xyz="0 0 0"/>
 		</visual>
 		<collision>
+			<origin rpy="-1.570796 3.141592 0" xyz="0 0 0"/>
 			<geometry>
-				<mesh filename="package://denso_vp6242_description/meshes/collision/link1.dae" scale="${scale_value*0.001} ${scale_value*0.001} ${scale_value*0.001}"/>
+				<mesh filename="package://denso_vp6242_description/meshes/collision/robot/link_1.dae" scale="${scale_value} ${scale_value} ${scale_value}"/>
 			</geometry>
-			<origin rpy="-1.570796 3.141592 0" xyz="0 0 0"/>
 		</collision>
 	</link>
-	<link name="link2">
+	<joint name="joint_1" type="revolute">
+		<parent link="base_link"/>
+		<child link="link_1" />
+		<origin rpy="0 0 0" xyz="0.0 0.0 ${scale_value*0.155}"/>
+		<axis xyz="0 0 1"/>
+		<limit effort="${scale_value * 1.0}" lower="-2.617994" upper="2.617994" velocity="${scale_value * 0.403171057210690}" />
+	</joint>
+	<link name="link_2">
 		<visual>
+			<origin rpy="-1.570796 3.141592 0" xyz="0 0 0"/>
 			<geometry>
-				<mesh filename="package://denso_vp6242_description/meshes/visual/link2.dae" scale="${scale_value*0.001} ${scale_value*0.001} ${scale_value*0.001}"/>
+				<mesh filename="package://denso_vp6242_description/meshes/visual/robot/link_2.dae" scale="${scale_value} ${scale_value} ${scale_value}"/>
 			</geometry>
-			<origin rpy="-1.570796 3.141592 0" xyz="0 0 0"/>
 		</visual>
 		<collision>
+			<origin rpy="-1.570796 3.141592 0" xyz="0 0 0"/>
 			<geometry>
-				<mesh filename="package://denso_vp6242_description/meshes/collision/link2.dae" scale="${scale_value*0.001} ${scale_value*0.001} ${scale_value*0.001}"/>
+				<mesh filename="package://denso_vp6242_description/meshes/collision/robot/link_2.dae" scale="${scale_value} ${scale_value} ${scale_value}"/>
 			</geometry>
-			<origin rpy="-1.570796 3.141592 0" xyz="0 0 0"/>
 		</collision>
 	</link>
-	<link name="link3">
+	<joint name="joint_2" type="revolute">
+		<parent link="link_1"/>
+		<child link="link_2"/>
+		<origin rpy="0 0 0" xyz="0.0 0.0 ${scale_value*0.125}"/>
+		<axis xyz="-0.000000 1.000000 -0.000000" />
+		<limit effort="${scale_value * 1.0}" lower="-1.047198" upper="1.745329" velocity="${scale_value * 0.392175482923126}" />
+	</joint>
+	<link name="link_3">
 		<visual>
+			<origin rpy="-1.570796 1.570796 0" xyz="0 0 0"/>
 			<geometry>
-				<mesh filename="package://denso_vp6242_description/meshes/visual/link3.dae" scale="${scale_value*0.001} ${scale_value*0.001} ${scale_value*0.001}"/>
+				<mesh filename="package://denso_vp6242_description/meshes/visual/robot/link_3.dae" scale="${scale_value} ${scale_value} ${scale_value}"/>
 			</geometry>
-			<origin rpy="-1.570796 1.570796 0" xyz="0 0 0"/>
 		</visual>
 		<collision>
+			<origin rpy="-1.570796 1.570796 0" xyz="0 0 0"/>
 			<geometry>
-				<mesh filename="package://denso_vp6242_description/meshes/collision/link3.dae" scale="${scale_value*0.001} ${scale_value*0.001} ${scale_value*0.001}"/>
+				<mesh filename="package://denso_vp6242_description/meshes/collision/robot/link_3.dae" scale="${scale_value} ${scale_value} ${scale_value}"/>
 			</geometry>
-			<origin rpy="-1.570796 1.570796 0" xyz="0 0 0"/>
 		</collision>
 	</link>
-	<link name="link4">
+	<joint name="joint_3" type="revolute">
+		<parent link="link_2"/>
+		<child link="link_3"/>
+		<origin rpy="0 0 0" xyz="0.0 0.0 ${scale_value*0.210}"/>
+		<axis xyz="-0.000000 1.000000 -0.000000" />
+		<limit effort="${scale_value * 1.0}" lower="0.3141593" upper="2.443461" velocity="${scale_value * 0.725707902979242}" />
+	</joint>
+	<link name="link_4">
 		<visual>
+			<origin rpy="0 1.570796 1.570796" xyz="0 0 ${scale_value*0.085}"/>
 			<geometry>
-				<mesh filename="package://denso_vp6242_description/meshes/visual/link4.dae" scale="${scale_value*0.001} ${scale_value*0.001} ${scale_value*0.001}"/>
+				<mesh filename="package://denso_vp6242_description/meshes/visual/robot/link_4.dae" scale="${scale_value} ${scale_value} ${scale_value}"/>
 			</geometry>
-			<origin rpy="0 1.570796 1.570796" xyz="0 0 ${scale_value*0.085}"/>
 		</visual>
 		<collision>
+			<origin rpy="0 1.570796 1.570796" xyz="0 0 ${scale_value*0.085}"/>
 			<geometry>
-				<mesh filename="package://denso_vp6242_description/meshes/collision/link4.dae" scale="${scale_value*0.001} ${scale_value*0.001} ${scale_value*0.001}"/>
+				<mesh filename="package://denso_vp6242_description/meshes/collision/robot/link_4.dae" scale="${scale_value} ${scale_value} ${scale_value}"/>
 			</geometry>
-			<origin rpy="0 1.570796 1.570796" xyz="0 0 ${scale_value*0.085}"/>
 		</collision>
 	</link>
-	<link name="link5">
+	<joint name="joint_4" type="revolute">
+		<parent link="link_3"/>
+		<child link="link_4"/>
+		<origin rpy="0 0 0" xyz="${scale_value*(-0.075)} 0.0 0.0"/>
+		<axis xyz="-0.000000 -0.000000 1.000000" />
+		<limit effort="${scale_value * 1.0}" lower="-2.96706" upper="2.96706" velocity="${scale_value * 0.739146938219599}" />
+	</joint>
+	<link name="link_5">
 		<visual>
+			<origin rpy="0 1.570796 1.570796" xyz="0 0 0.0"/>
 			<geometry>
-				<mesh filename="package://denso_vp6242_description/meshes/visual/link5.dae" scale="${scale_value*0.001} ${scale_value*0.001} ${scale_value*0.001}"/>
+				<mesh filename="package://denso_vp6242_description/meshes/visual/robot/link_5.dae" scale="${scale_value} ${scale_value} ${scale_value}"/>
 			</geometry>
-			<origin rpy="0 1.570796 1.570796" xyz="0 0 0.0"/>
 		</visual>
 		<collision>
+			<origin rpy="0 1.570796 1.570796" xyz="0 0 0.0"/>
 			<geometry>
-				<mesh filename="package://denso_vp6242_description/meshes/collision/link5.dae" scale="${scale_value*0.001} ${scale_value*0.001} ${scale_value*0.001}"/>
+				<mesh filename="package://denso_vp6242_description/meshes/collision/robot/link_5.dae" scale="${scale_value} ${scale_value} ${scale_value}"/>
 			</geometry>
-			<origin rpy="0 1.570796 1.570796" xyz="0 0 0.0"/>
 		</collision>
 	</link>
-	<link name="link6">
+	<joint name="joint_5" type="revolute">
+		<parent link="link_4"/>
+		<child link="link_5"/>
+		<origin rpy="0 0 0" xyz="0.0 0.0 ${scale_value*0.210}"/>
+		<axis xyz="-0.000000 1.000000 -0.000000" />
+		<limit effort="${scale_value * 1.0}" lower="-1.658063" upper="2.356194" velocity="${scale_value * 0.739146938219599}" />
+	</joint>
+	<link name="link_6">
 		<visual>
 			<geometry>
@@ -108,179 +145,13 @@
 		</collision>
 	</link>
-	<link name="tool0"/>
-	<!-- Joint list -->
-	<joint name="joint1" type="revolute">
-		<origin rpy="0 0 0" xyz="0.0 0.0 ${scale_value*0.155}"/>
-		<parent link="base_link"/>
-		<child link="link1"/>
-		<axis xyz="0 0 1"/>
-		<limit effort="100000" lower="-2.792526803" upper="2.792526803" velocity="4.36332312999"/>
+	<joint name="joint_6" type="revolute">
+		<parent link="link_5"/>
+		<child link="link_6"/>
+		<origin rpy="0 0 0" xyz="0.0 0.0 ${scale_value*0.07}"/>
+		<axis xyz="-0.000000 -0.000000 1.000000" />
+		<limit effort="${scale_value * 1.0}" lower="-2.96706" upper="2.96706" velocity="${scale_value * 1.109331272567600}" />
 	</joint>
-	<joint name="joint2" type="revolute">
-		<origin rpy="0 0 0" xyz="0.0 0.0 ${scale_value*0.125}"/>
-		<parent link="link1"/>
-		<child link="link2"/>
-		<axis xyz="0 1 0"/>
-		<limit effort="100000" lower="-2.094395102" upper="2.094395102" velocity="3.26376570123"/>
-	</joint>
-		<joint name="joint3" type="revolute">
-		<origin rpy="0 0 0" xyz="0.0 0.0 ${scale_value*0.210}"/>
-		<parent link="link2"/>
-		<child link="link3"/>
-		<axis xyz="0 1 0"/>
-		<limit effort="100000" lower="0.331612558" upper="2.792526803" velocity="4.36332312999"/>
-	</joint>
-	<joint name="joint4" type="revolute">
-		<origin rpy="0 0 0" xyz="${scale_value*(-0.075)} 0.0 0.0"/>
-		<parent link="link3"/>
-		<child link="link4"/>
-		<axis xyz="0 0 1"/>
-		<limit effort="100000" lower="-2.792526803" upper="2.792526803" velocity="5.23598775598"/>
-	</joint>
-	<joint name="joint5" type="revolute">
-		<origin rpy="0 0 0" xyz="0.0 0.0 ${scale_value*0.210}"/>
-		<parent link="link4"/>
-		<child link="link5"/>
-		<axis xyz="0 1 0"/>
-		<limit effort="100000" lower="-2.094395102" upper="2.094395102" velocity="5.23598775598"/>
-	</joint>
-	<joint name="joint6" type="revolute">
-		<origin rpy="0 0 0" xyz="0.0 0.0 ${scale_value*0.07}"/>
-		<parent link="link5"/>
-		<child link="link6"/>
-		<axis xyz="0 0 1"/>
-		<limit effort="100000" lower="-3.14159265359" upper="3.14159265359" velocity="5.23598775598"/>
-	</joint>
-	<joint name="joint6-tool0" type="fixed">
-		<parent link="link6"/>
-		<child link="tool0"/>
-		<origin rpy="0 0 0" xyz="0 0 0"/>
-  	</joint>
-	<link name="robot_gripper_interface1">
-		<collision>
-			<origin rpy="0 0 0" xyz="0 0 ${scale_value*0.0045}"/>
-			<geometry>
-				<cylinder length="${scale_value*0.009}" radius="${scale_value*0.04}"/>
-			</geometry>
-		</collision>
-		<visual>
-			<origin rpy="0 0 0" xyz="0 0 ${scale_value*0.0045}"/>
-			<geometry>
-				<cylinder length="${scale_value*0.009}" radius="${scale_value*0.04}"/>
-			</geometry>
-			<material name="material_color_robot_gripper_interface1">
-				<color rgba="0.6 1 0.6 1"/>
-			</material>
-		</visual>
-	</link>
-	<link name="robot_gripper_interface2">
-		<collision>
-			<origin rpy="0 0 0" xyz="0 0 ${scale_value*0.0045}"/>
-			<geometry>
-				<cylinder length="${scale_value*0.009}" radius="${scale_value*0.04}"/>
-			</geometry>
-		</collision>
-		<visual>
-			<origin rpy="0 0 0" xyz="0 0 ${scale_value*0.0045}"/>
-			<geometry>
-				<cylinder length="${scale_value*0.009}" radius="${scale_value*0.04}"/>
-			</geometry>
-			<material name="material_color_robot_gripper_interface2">
-				<color rgba="0.6 1 0.6 1"/>
-			</material>
-		</visual>
-	</link>
-	<link name="gripper_body">
-		<collision>
-			<origin rpy="0 0 0" xyz="0 0 ${scale_value*0.042}"/>
-			<geometry>
-				<box size="${scale_value*0.11} ${scale_value*0.04} ${scale_value*0.084}"/>
-			</geometry>
-		</collision>
-		<visual>
-			<origin rpy="0 0 0" xyz="0 0 ${scale_value*0.042}"/>
-			<geometry>
-				<box size="${scale_value*0.11} ${scale_value*0.04} ${scale_value*0.084}"/>
-			</geometry>
-			<material name="material_color_gripper_body">
-				<color rgba="0.2 0.2 0.2 1"/>
-			</material>
-		</visual>
-	</link>
-	<link name="right_claw">
-		<collision>
-			<origin rpy="0 0 0" xyz="0 0 ${scale_value*0.0068}"/>
-			<geometry>
-				<box size="${scale_value*0.05075} ${scale_value*0.015} ${scale_value*0.0136}"/>
-			</geometry>
-		</collision>
-		<visual>
-			<origin rpy="0 0 0" xyz="0 0 ${scale_value*0.0068}"/>
-			<geometry>
-				<box size="${scale_value*0.05075} ${scale_value*0.015} ${scale_value*0.0136}"/>
-			</geometry>
-			<material name="material_color_right_claw">
-				<color rgba="0.6 0.6 1 1"/>
-			</material>
-		</visual>
-	</link>
-	<link name="left_claw">
-		<collision>
-			<origin rpy="0 0 0" xyz="0 0 ${scale_value*0.0068}"/>
-			<geometry>
-				<box size="${scale_value*0.05075} ${scale_value*0.015} ${scale_value*0.0136}"/>
-			</geometry>
-		</collision>
-		<visual>
-		<origin rpy="0 0 0" xyz="0 0 ${scale_value*0.0068}"/>
-			<geometry>
-				<box size="${scale_value*0.05075} ${scale_value*0.015} ${scale_value*0.0136}"/>
-			</geometry>
-			<material name="material_color_left_claw">
-				<color rgba="0.6 0.6 1 1"/>
-			</material>
-		</visual>
-	</link>
-	<link name="peak_tool"/>
-	<!--joint of robot and gripper interface-->
-	<joint name="robot_to_gripper" type="fixed">
-		<parent link="tool0"/>
-		<child link="robot_gripper_interface1"/>
-		<origin rpy="0 0 1.57079632679" xyz="0 0 0"/>
-	</joint>
-	<!--joint of gripper interface and body-->
-	<joint name="robot_to_gripper_interface_2" type="fixed">
-		<parent link="robot_gripper_interface1"/>
-		<child link="robot_gripper_interface2"/>
-		<origin rpy="0 0 0" xyz="0 0 ${scale_value*0.009}"/>
-	</joint>
-	<joint name="interface_to_gripper_body" type="fixed">
-		<parent link="robot_gripper_interface2"/>
-		<child link="gripper_body"/>
-		<origin rpy="0 0 0" xyz="0.0 0.0 ${scale_value*0.009}"/>
-	</joint>
-	<!--joint of gripper and claw-->
-	<joint name="right_claw_joint" type="prismatic">
-		<parent link="gripper_body"/>
-		<child link="right_claw"/>
-		<origin rpy="0.000000 0.000000 0.000000" xyz="${scale_value*0.029625} 0 ${scale_value*0.084}"/>
-		<axis xyz="1.000000 0.000000 -0.000000"/>
-		<limit effort="${scale_value * 200000}" lower="-${scale_value * 0.0015000}" upper="0.0" velocity="0.1"/>
-		<dynamics damping="0" friction="0"/>
-	</joint>
-	<joint name="left_claw_joint" type="prismatic">
-		<parent link="gripper_body"/>
-		<child link="left_claw"/>
-		<mimic joint="right_claw_joint" multiplier="-1.000000" offset="0.000000"/>
-		<origin rpy="0.000000 0.000000 0.000000" xyz="${scale_value*(-0.029625)} 0 ${scale_value*0.084}"/>
-		<axis xyz="1.000000 0.000000 -0.000000"/>
-		<limit effort="${scale_value * 200000}" lower="0.0" upper="${scale_value * (0.00150000)}" velocity="0.1"/>
-		<dynamics damping="0" friction="0"/>
-	</joint>
-	<!--joint of gripper and peak tool-->
-	<joint name="peak_tool" type="fixed">
-		<origin rpy="0 3.14159265359 0" xyz="0 0 ${scale_value*0.0976}"/>
-		<parent link="gripper_body"/>
-		<child link="peak_tool"/>
-	</joint>
+	<xacro:if value="${gripper_type != 'none'}">
+		<xacro:include filename="$(find denso_vp6242_description)/urdf/${gripper_type}.urdf.xacro" />
+	</xacro:if>
 </robot>

File: ROS2_ws/src/denso_vp6242_moveit_config/config/denso_vp6242.ros2_control.xacro (robot description, xacro)
@@ -8,50 +8,50 @@
                 <plugin>mock_components/GenericSystem</plugin>
             </hardware>
-            <joint name="joint1">
+            <joint name="joint_1">
                 <command_interface name="position"/>
                 <state_interface name="position">
-                  <param name="initial_value">${initial_positions['joint1']}</param>
+                  <param name="initial_value">${initial_positions['joint_1']}</param>
                 </state_interface>
                 <state_interface name="velocity"/>
             </joint>
-            <joint name="joint2">
+            <joint name="joint_2">
                 <command_interface name="position"/>
                 <state_interface name="position">
-                  <param name="initial_value">${initial_positions['joint2']}</param>
+                  <param name="initial_value">${initial_positions['joint_2']}</param>
                 </state_interface>
                 <state_interface name="velocity"/>
             </joint>
-            <joint name="joint3">
+            <joint name="joint_3">
                 <command_interface name="position"/>
                 <state_interface name="position">
-                  <param name="initial_value">${initial_positions['joint3']}</param>
+                  <param name="initial_value">${initial_positions['joint_3']}</param>
                 </state_interface>
                 <state_interface name="velocity"/>
             </joint>
-            <joint name="joint4">
+            <joint name="joint_4">
                 <command_interface name="position"/>
                 <state_interface name="position">
-                  <param name="initial_value">${initial_positions['joint4']}</param>
+                  <param name="initial_value">${initial_positions['joint_4']}</param>
                 </state_interface>
                 <state_interface name="velocity"/>
             </joint>
-            <joint name="joint5">
+            <joint name="joint_5">
                 <command_interface name="position"/>
                 <state_interface name="position">
-                  <param name="initial_value">${initial_positions['joint5']}</param>
+                  <param name="initial_value">${initial_positions['joint_5']}</param>
                 </state_interface>
                 <state_interface name="velocity"/>
             </joint>
-            <joint name="joint6">
+            <joint name="joint_6">
                 <command_interface name="position"/>
                 <state_interface name="position">
-                  <param name="initial_value">${initial_positions['joint6']}</param>
+                  <param name="initial_value">${initial_positions['joint_6']}</param>
                 </state_interface>
                 <state_interface name="velocity"/>
             </joint>
-            <joint name="right_claw_joint">
+            <joint name="joint_gripper">
                 <command_interface name="position"/>
                 <state_interface name="position">
-                  <param name="initial_value">${initial_positions['right_claw_joint']}</param>
+                  <param name="initial_value">${initial_positions['joint_gripper']}</param>
                 </state_interface>
                 <state_interface name="velocity"/>

Commit message: Several changes to reestructure how the robot joint trajectories were created

File: ROS2_ws/src/denso_vp6242_description/urdf/denso_vp6242.urdf.xacro (robot description, xacro)
@@ -4,9 +4,4 @@
 	<xacro:property name="gripper_type" value="$(arg gripper_type)" />
 	<xacro:property name="scale_value" value="100.0"/>
-	<link name="world"/>
-	<joint name="joint_w" type="fixed">
-		<parent link="world"/>
-		<child link="base_link"/>
-	</joint>
 	<link name="base_link">
 		<visual>
@@ -42,5 +37,5 @@
 		<origin rpy="0 0 0" xyz="0.0 0.0 ${scale_value*0.155}"/>
 		<axis xyz="0 0 1"/>
-		<limit effort="${scale_value * 1.0}" lower="-2.617994" upper="2.617994" velocity="${scale_value * 0.403171057210690}" />
+		<limit effort="${scale_value * 100.0}" lower="-2.792526803" upper="2.792526803" velocity="0.403171057210690"/>
 	</joint>
 	<link name="link_2">
@@ -63,5 +58,5 @@
 		<origin rpy="0 0 0" xyz="0.0 0.0 ${scale_value*0.125}"/>
 		<axis xyz="-0.000000 1.000000 -0.000000" />
-		<limit effort="${scale_value * 1.0}" lower="-1.047198" upper="1.745329" velocity="${scale_value * 0.392175482923126}" />
+		<limit effort="${scale_value * 100.0}" lower="-2.094395102" upper="2.094395102" velocity="0.392175482923126" />
 	</joint>
 	<link name="link_3">
@@ -84,5 +79,5 @@
 		<origin rpy="0 0 0" xyz="0.0 0.0 ${scale_value*0.210}"/>
 		<axis xyz="-0.000000 1.000000 -0.000000" />
-		<limit effort="${scale_value * 1.0}" lower="0.3141593" upper="2.443461" velocity="${scale_value * 0.725707902979242}" />
+		<limit effort="${scale_value * 100.0}" lower="0.331612558" upper="2.792526803" velocity="0.725707902979242" />
 	</joint>
 	<link name="link_4">
@@ -105,5 +100,5 @@
 		<origin rpy="0 0 0" xyz="${scale_value*(-0.075)} 0.0 0.0"/>
 		<axis xyz="-0.000000 -0.000000 1.000000" />
-		<limit effort="${scale_value * 1.0}" lower="-2.96706" upper="2.96706" velocity="${scale_value * 0.739146938219599}" />
+		<limit effort="${scale_value * 100.0}" lower="-2.792526803" upper="2.792526803" velocity="0.739146938219599" />
 	</joint>
 	<link name="link_5">
@@ -126,5 +121,5 @@
 		<origin rpy="0 0 0" xyz="0.0 0.0 ${scale_value*0.210}"/>
 		<axis xyz="-0.000000 1.000000 -0.000000" />
-		<limit effort="${scale_value * 1.0}" lower="-1.658063" upper="2.356194" velocity="${scale_value * 0.739146938219599}" />
+		<limit effort="${scale_value * 100.0}" lower="-2.094395102" upper="2.094395102" velocity="0.739146938219599" />
 	</joint>
 	<link name="link_6">
@@ -138,10 +133,4 @@
 			</material>
 		</visual>
-		<collision>
-			<geometry>
-				<cylinder length="${scale_value*0.01}" radius="${scale_value*0.0205}"/>
-			</geometry>
-			<origin rpy="0 0 0" xyz="0.0 0.0 ${scale_value*(-0.005)}"/>
-		</collision>
 	</link>
 	<joint name="joint_6" type="revolute">
@@ -150,5 +139,5 @@
 		<origin rpy="0 0 0" xyz="0.0 0.0 ${scale_value*0.07}"/>
 		<axis xyz="-0.000000 -0.000000 1.000000" />
-		<limit effort="${scale_value * 1.0}" lower="-2.96706" upper="2.96706" velocity="${scale_value * 1.109331272567600}" />
+		<limit effort="${scale_value * 100.0}" lower="-2.96706" upper="2.96706" velocity="1.109331272567600" />
 	</joint>
 	<xacro:if value="${gripper_type != 'none'}">
