Commit message: Added new gripper to the epson t3 robot (#27)
* Added new gripper to the epson t3 robot

* changed the config file for the epson t3 and the support for epson t3 to the task_client_action_server added with proper gripper options.

* removed additional file "task_creator_action_server_bkup.cpp"

* Added the new dog plan (the one that works)

* Delete oneblock.csv

---------

Co-authored-by: bexprove <rakshithbasakr@gmail.com>
Co-authored-by: Pedro Saman <pedrosaman96@gmail.com>

File: ROS2_ws/src/epson_t3_description/urdf/epson_t3_description.urdf.xacro (robot description, xacro)
@@ -1,7 +1,14 @@
 <?xml version="1.0" encoding="utf-8"?>
 <robot name="epson_t3" xmlns:xacro="http://www.ros.org/wiki/xacro">
-  <xacro:arg name="gripper_type" default="tayo"/>
+  <xacro:arg name="gripper_type" default="taiyo_sd_2005"/>
 	<xacro:property name="gripper_type" value="$(arg gripper_type)" />
 	<xacro:property name="scale_value" value="100.0"/>
+  <xacro:property name="scale_value1" value="0.2"/>
+  <link name="world"/>
+  <joint name="joint_w" type="fixed">
+    <parent link="world"/>
+    <child link="base_link"/>
+    <origin rpy="0.0 0.0 0.0" xyz="-10 0 26"/>
+  </joint>
   <link name="base_link">
     <visual>
@@ -60,5 +67,5 @@
   <link name="link_3">
     <visual>
-      <origin xyz="0 0 0" rpy="0 0 0" />
+      <origin xyz="0 ${scale_value*0.32} 0" rpy="0 0 0" /> <!--Changed the Y-axis-->
       <geometry>
         <mesh filename="package://epson_t3_description/meshes/link_3.STL" scale="${scale_value} ${scale_value} ${scale_value}"/>
@@ -70,5 +77,5 @@
     </visual>
     <collision>
-      <origin xyz="0 0 0" rpy="0 0 0" />
+      <origin xyz="0 ${scale_value*0.32} 0" rpy="0 0 0" /> <!--Changed the Y-axis-->
       <geometry>
         <mesh filename="package://epson_t3_description/meshes/link_3.STL" scale="${scale_value} ${scale_value} ${scale_value}"/>
@@ -91,15 +98,15 @@
   </joint>
   <joint name="joint_3" type="prismatic">
-    <origin xyz="${scale_value*0.175} ${scale_value*0} 0" rpy="0 1.0337 0" />
+    <origin xyz="${scale_value*0.175} 0 0" rpy="0 1.0337 0" />
     <parent link="link_2" />
     <child link="link_2_virtual" />
     <axis xyz="0 1 0" />
-    <limit lower="${scale_value*-0.1200}" upper="${scale_value*-0.0220}" effort="10" velocity="0.1" />
+    <limit lower="${scale_value*-0.11949}" upper="${scale_value*-0.042}" effort="10" velocity="1" /> <!--changed the limits-->
   </joint>
   <joint name="joint_4" type="revolute">
-    <origin xyz="0 0 0" rpy="0 0 -3.14" />
+    <origin xyz="0 0 0" rpy="0 0 0" /> <!--Increased Y-axis by 0.22-->
     <parent link="link_2_virtual" />
     <child link="link_3" />
-    <axis xyz="0 1 0" />
+    <axis xyz="0 1 0"/>
     <limit lower="-3.14" upper="3.14" effort="0" velocity="0" />
   </joint>
@@ -107,9 +114,3 @@
    	<xacro:include filename="$(find epson_t3_description)/urdf/${gripper_type}.urdf.xacro" />
   </xacro:if>
-  <link name="world"/>
-  <joint name="fixed" type="fixed">
-    <parent link="world"/>
-    <child link="base_link"/>
-    <origin xyz="-10 0 20"/>
-  </joint>
 </robot>

File: ROS2_ws/src/epson_t3_description/urdf/taiyo.urdf.xacro (robot description, xacro)
@@ -8,5 +8,5 @@
 			</geometry>
 		</visual>
-		<collision>
+		<collision>7222
 			<origin rpy="0 0 1.57079632679" xyz="0 0 ${scale_value*0.042135}"/>
 			<geometry>
@@ -40,5 +40,5 @@
 		<parent link="link_3"/>
 		<child link="robot_gripper_interface"/>
-		<origin rpy="-1.5708 0 0" xyz="0 1 0"/>
+		<origin rpy="1.5708 3.14159 0" xyz="0 0 0"/> <!--DECREASED Y-Axis from orign-->
 	</joint>
 	<joint name="joint_gripper_base" type="fixed">
